File: cp2102-esp32-autoprogram.kicad_sch (KiCad schematic)
At the start: 7 parts, among them Q401 MMDT3904, U401 CP2102-GMR

Commit message: add mouser part numbers
Parts:
- C401, C403: Mouser (none) -> 581-06035C104KAT2A
- C402: Mouser (none) -> 603-CC603KRX5R8BB105
- Q401: Mouser (none) -> 621-MMDT3904-F
- R401, R402: Mouser (none) -> 603-RC0603FR-0710KL
- U401: Mouser (none) -> 634-CP2102-GMR
Changed lines of the file:
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@@
+      (effects (font (size 1.27 1.27)) hide)
+    )
+    (property "Mouser" "603-RC0603FR-0710KL" (at 132.08 30.48 0)
       (effects (font (size 1.27 1.27)) hide)
     )
@@
     )
     (property "LCSC" "C6568" (at 66.04 67.31 0)
+      (effects (font (size 1.27 1.27)) hide)
+    )
+    (property "Mouser" "634-CP2102-GMR" (at 66.04 67.31 0)
       (effects (font (size 1.27 1.27)) hide)
     )
@@
       (effects (font (size 1.27 1.27)) hide)
     )
+    (property "Mouser" "581-06035C104KAT2A" (at 33.02 41.91 0)
+      (effects (font (size 1.27 1.27)) hide)
+    )
     (pin "1")
     (pin "2")
@@
       (effects (font (size 1.27 1.27)) hide)
     )
+    (property "Mouser" "603-RC0603FR-0710KL" (at 132.08 48.26 0)
+      (effects (font (size 1.27 1.27)) hide)
+    )
     (pin "1")
     (pin "2")
@@
     )
     (property "LCSC" "C14663" (at 21.59 41.91 0)
+      (effects (font (size 1.27 1.27)) hide)
+    )
+    (property "Mouser" "603-CC603KRX5R8BB105" (at 21.59 41.91 0)
       (effects (font (size 1.27 1.27)) hide)
     )
@@
     )
     (property "LCSC" " C83572" (at 143.51 48.26 0)
+      (effects (font (size 1.27 1.27)) hide)
+    )
+    (property "Mouser" "621-MMDT3904-F" (at 143.51 48.26 0)
       (effects (font (size 1.27 1.27)) hide)
     )
@@
       (effects (font (size 1.27 1.27)) hide)
     )
+    (property "Mouser" "621-MMDT3904-F" (at 143.51 30.48 0)
+      (effects (font (size 1.27 1.27)) hide)
+    )
     (pin "1")
     (pin "2")
@@
       (effects (font (size 1.27 1.27)) hide)
     )
+    (property "Mouser" "581-06035C104KAT2A" (at 93.98 31.75 0)
+      (effects (font (size 1.27 1.27)) hide)
+    )
